File: PCB-Design/IoT.brd (EAGLE design)
At the start: 60.9 x 56.8 mm, 11 parts, among them M2 ARDUINO-NANO-3.0, M3 WIRELESS-NRF24L01

Commit message: more branding
Other:
- board size 60.9 x 56.8 mm -> 60.9 x 55.5 mm
- board text added: "School of Electrical and Information Engineering"
Changed lines of the file:
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@@
 <grid distance="50" unitdist="mil" unit="mm" style="dots" multiple="1" display="yes" altdistance="5" altunitdist="mil" altunit="mm"/>
 <layers>
-<layer number="1" name="Top" color="4" fill="1" visible="no" active="yes"/>
+<layer number="1" name="Top" color="4" fill="1" visible="yes" active="yes"/>
 <layer number="2" name="Route2" color="16" fill="1" visible="no" active="no"/>
 <layer number="3" name="Route3" color="17" fill="1" visible="no" active="no"/>
@@
 <layer number="14" name="Route14" color="22" fill="1" visible="no" active="no"/>
 <layer number="15" name="Route15" color="23" fill="1" visible="no" active="no"/>
-<layer number="16" name="Bottom" color="1" fill="1" visible="no" active="yes"/>
+<layer number="16" name="Bottom" color="1" fill="1" visible="yes" active="yes"/>
 <layer number="17" name="Pads" color="2" fill="1" visible="yes" active="yes"/>
-<layer number="18" name="Vias" color="2" fill="1" visible="no" active="yes"/>
-<layer number="19" name="Unrouted" color="6" fill="1" visible="no" active="yes"/>
-<layer number="20" name="Dimension" color="24" fill="1" visible="no" active="yes"/>
+<layer number="18" name="Vias" color="2" fill="1" visible="yes" active="yes"/>
+<layer number="19" name="Unrouted" color="6" fill="1" visible="yes" active="yes"/>
+<layer number="20" name="Dimension" color="24" fill="1" visible="yes" active="yes"/>
 <layer number="21" name="tPlace" color="7" fill="1" visible="yes" active="yes"/>
 <layer number="22" name="bPlace" color="7" fill="1" visible="no" active="yes"/>
-<layer number="23" name="tOrigins" color="15" fill="1" visible="no" active="yes"/>
+<layer number="23" name="tOrigins" color="15" fill="1" visible="yes" active="yes"/>
 <layer number="24" name="bOrigins" color="15" fill="1" visible="no" active="yes"/>
 <layer number="25" name="tNames" color="7" fill="1" visible="no" active="yes"/>
@@
 <layer number="47" name="Measures" color="7" fill="1" visible="no" active="yes"/>
 <layer number="48" name="Document" color="7" fill="1" visible="no" active="yes"/>
-<layer number="49" name="Reference" color="7" fill="1" visible="yes" active="yes"/>
+<layer number="49" name="Reference" color="7" fill="1" visible="no" active="yes"/>
 <layer number="50" name="dxf" color="7" fill="1" visible="no" active="no"/>
 <layer number="51" name="tDocu" color="7" fill="1" visible="yes" active="yes"/>
@@
 <board>
 <plain>
-<wire x1="-2.54" y1="44.45" x2="58.4" y2="44.45" width="0" layer="20"/>
-<wire x1="58.4" y1="44.45" x2="58.4" y2="101.27" width="0" layer="20"/>
+<wire x1="-2.54" y1="45.72" x2="58.4" y2="45.72" width="0" layer="20"/>
+<wire x1="58.4" y1="45.72" x2="58.4" y2="101.27" width="0" layer="20"/>
 <wire x1="58.4" y1="101.27" x2="-2.54" y2="101.27" width="0" layer="20"/>
-<wire x1="-2.54" y1="101.27" x2="-2.54" y2="44.45" width="0" layer="20"/>
+<wire x1="-2.54" y1="101.27" x2="-2.54" y2="45.72" width="0" layer="20"/>
 <dimension x1="-2.54" y1="52.07" x2="58.42" y2="52.07" x3="27.94" y3="26.67" textsize="1.778" layer="1"/>
 <dimension x1="-1.27" y1="105.41" x2="-1.27" y2="44.45" x3="-17.78" y3="74.93" textsize="1.778" layer="1"/>
-<text x="6.35" y="46.99" size="2.54" layer="51" font="vector" rot="R90">Wits ParkSmart
+<text x="6.35" y="48.26" size="2.54" layer="51" font="vector" rot="R90">Wits ParkSmart
 2018</text>
+<dimension x1="-2.54" y1="101.6" x2="-2.54" y2="44.45" x3="-8.89" y3="73.025" textsize="1.778" layer="16"/>
+<text x="55.88" y="48.26" size="1.3" layer="51" font="vector" align="bottom-right">School of Electrical and Information Engineering</text>
 </plain>
 <attributes>
