File: PCB-Design/GatewayNode.brd (EAGLE design)
At the start: 60.9 x 55.5 mm, 11 parts, among them M3 WIRELESS-NRF24L01

Commit message: final gateway node PCB design
Parts:
- removed HC-SR04-2, HC-SR04-3, HC-SR04-4: ULTRASONIC-HC-SR04#V, diy-modules:ULTRASONIC-HC-SR04#V
- moved U$1 70.3 mm to (34.3, 64.8), turned to 90 degrees
- moved HC-SR04-1 41.7 mm to (49.5, 81.3)
- moved U$6 19.7 mm to (24.1, 83.8)
- moved C1 3.81 mm to (24.1, 87.6)
- moved R1 3.81 mm to (19.1, 92.7)
- moved C2 2.54 mm to (24.1, 96.5)
- moved M3 1.27 mm to (43.2, 90.2)
Connections:
- removed net N$11: HC-SR04-3.2
- removed net N$12: HC-SR04-4.3
- removed net N$13: HC-SR04-4.2
- removed net N$14: M3.3
- removed net N$15: M3.4
- removed net N$16: M3.5
- removed net N$17: M3.6
- removed net N$18: M3.7
- new net N$3: M3.3, U$1.D4
- new net N$4: M3.5, U$1.D5
- net GND: now also U$1.GND@0, U$1.GND@1, U$1.GND@2, U$1.GND@3
- net N$1: now also U$1.D3
- net N$10: now also HC-SR04-1.3, U$1.D1; no longer HC-SR04-3.3
- net N$2: now also U$1.3V3@1
- net N$5: now also M3.7, U$1.D6; no longer HC-SR04-1.2
- net N$6: now also M3.4, U$1.D8; no longer HC-SR04-1.3
- net N$7: now also M3.6, U$1.D7; no longer HC-SR04-2.3
- net N$8: now also HC-SR04-1.2, U$1.D0; no longer HC-SR04-2.2
- net N$9: no longer HC-SR04-2.4, HC-SR04-3.4, HC-SR04-4.4
- net VCC: now also U$1.VIN; no longer HC-SR04-2.1, HC-SR04-3.1, HC-SR04-4.1
Routing:
- net N$8: track 6.66 -> 127.0 mm
- net N$9: track 140.4 -> 45.5 mm
- net N$10: track 3.81 -> 80.7 mm
- net N$15: track 46.2 -> 0.00 mm
- net N$17: track 42.9 -> 0.00 mm
- net N$3: track 0.00 -> 35.9 mm
- net N$18: track 33.5 -> 0.00 mm
- net N$1: track 46.0 -> 14.8 mm
- net N$16: track 30.1 -> 0.00 mm
- net N$4: track 0.00 -> 20.4 mm
- net N$14: track 16.6 -> 0.00 mm
- net N$13: track 13.3 -> 0.00 mm
- net N$7: track 6.66 -> 19.3 mm
- net VCC: track 98.3 -> 87.0 mm
- net N$12: track 11.0 -> 0.00 mm
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