File: PCB-Design/GatewayNode.sch (EAGLE design)
At the start: 11 parts, among them M3 WIRELESS-NRF24L01

Commit message: final gateway node PCB design
Parts:
- removed HC-SR04-2, HC-SR04-3, HC-SR04-4: ULTRASONIC-HC-SR04#V, diy-modules:ULTRASONIC-HC-SR04#V
Connections:
- removed net N$11: HC-SR04-3.TRIG
- removed net N$12: HC-SR04-4.ECHO
- removed net N$13: HC-SR04-4.TRIG
- removed net N$14: M3.CE
- removed net N$15: M3.CSN
- removed net N$16: M3.SCK
- removed net N$17: M3.MOSI
- removed net N$18: M3.MISO
- new net N$3: M3.CE, U$1.D4
- new net N$4: M3.SCK, U$1.D5
- net GND: now also U$1.GND@0, U$1.GND@1, U$1.GND@2, U$1.GND@3
- net N$1: now also U$1.D3
- net N$10: now also HC-SR04-1.ECHO, U$1.D1; no longer HC-SR04-3.ECHO
- net N$2: now also U$1.3V3@1
- net N$5: now also M3.MISO, U$1.D6; no longer HC-SR04-1.TRIG
- net N$6: now also M3.CSN, U$1.D8; no longer HC-SR04-1.ECHO
- net N$7: now also M3.MOSI, U$1.D7; no longer HC-SR04-2.ECHO
- net N$8: now also HC-SR04-1.TRIG, U$1.D0; no longer HC-SR04-2.TRIG
- net N$9: no longer HC-SR04-2.GND, HC-SR04-3.GND, HC-SR04-4.GND
- net VCC: now also U$1.VIN; no longer HC-SR04-2.VCC, HC-SR04-3.VCC, HC-SR04-4.VCC
Other:
- moved on the sheet: HC-SR04-1, M3, U$1
